File: PCB/farmBot PCB3 v23.brd (EAGLE design)
At the start: 53.3 x 59.7 mm, 9 parts

Commit message: new pcb
Parts:
- moved DIGITAL_IN 30.9 mm to (18.5, 61.0)
- moved ANALOG_IN 26.7 mm to (53.3, 59.7)
Routing:
- net LIGHT0: track 44.8 -> 0.00 mm
- net LIGHT1: track 42.3 -> 0.00 mm
- net GND: track 157.7 -> 192.6 mm, vias 0 -> 3
- net D2: track 39.1 -> 6.37 mm
- net A3: track 33.7 -> 6.13 mm, vias 1 -> 0
- net A2: track 32.4 -> 8.78 mm, vias 1 -> 0
- net D6: track 29.5 -> 16.8 mm
- net D7: track 31.0 -> 20.4 mm
- net SDL: track 60.5 -> 51.7 mm, vias 1 -> 3
- net D8: track 32.9 -> 24.5 mm
- net 5V: track 113.8 -> 121.1 mm
- net SDA: track 55.3 -> 48.4 mm, vias 1 -> 5
- net D9: track 34.4 -> 28.1 mm
- net A1: track 16.9 -> 22.6 mm, vias 0 -> 2
- net PUMP: track 51.0 -> 45.4 mm
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